File: hardware/board/dc25-darknet-dialer.sch (EAGLE design)
At the start: 61 parts

Commit message: Updated board to include values for bypass caps
Parts:
- added C16: 4.7uF, SYNShop:C-USC0603
- C12, C13, C14: value (none) -> 100nF
- C15: value (none) -> 10nF
Connections:
- net GND: now also C16.1
- net VCC: now also C16.2
Changed lines of the file:
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@@
 <part name="U$8" library="SYNShop" deviceset="VCC" device=""/>
 <part name="U$9" library="SYNShop" deviceset="VCC" device=""/>
-<part name="C12" library="SYNShop" deviceset="C-US" device="C0603"/>
-<part name="C13" library="SYNShop" deviceset="C-US" device="C0603"/>
-<part name="C14" library="SYNShop" deviceset="C-US" device="C0603"/>
-<part name="C15" library="SYNShop" deviceset="C-US" device="C0603"/>
+<part name="C12" library="SYNShop" deviceset="C-US" device="C0603" value="100nF"/>
+<part name="C13" library="SYNShop" deviceset="C-US" device="C0603" value="100nF"/>
+<part name="C14" library="SYNShop" deviceset="C-US" device="C0603" value="100nF"/>
+<part name="C15" library="SYNShop" deviceset="C-US" device="C0603" value="10nF"/>
 <part name="GND21" library="SYNShop" deviceset="GND" device=""/>
 <part name="U$10" library="SYNShop" deviceset="VCC" device=""/>
+<part name="C16" library="SYNShop" deviceset="C-US" device="C0603" value="4.7uF"/>
 </parts>
 <sheets>
@@
 <instance part="GND21" gate="1" x="114.3" y="134.62"/>
 <instance part="U$10" gate="G$1" x="114.3" y="144.78"/>
+<instance part="C16" gate="G$1" x="73.66" y="139.7" rot="R180"/>
 </instances>
 <busses>
@@
 <junction x="93.98" y="137.16"/>
 <junction x="104.14" y="137.16"/>
+<pinref part="C16" gate="G$1" pin="1"/>
+<wire x1="83.82" y1="137.16" x2="73.66" y2="137.16" width="0.1524" layer="91"/>
+<junction x="83.82" y="137.16"/>
 </segment>
 </net>
@@
 <pinref part="U$10" gate="G$1" pin="VCC"/>
 <junction x="114.3" y="144.78"/>
-</segment>
-</net>
+<pinref part="C16" gate="G$1" pin="2"/>
+<wire x1="83.82" y1="144.78" x2="73.66" y2="144.78" width="0.1524" layer="91"/>
+<junction x="83.82" y="144.78"/>
+</segment>
+</net>

Commit message: Routing and layout progress
Connections:
- net N$38 renamed OLED_SPI_NSS
- new net N$38: U$2.PF0
- new net N$39: U$2.PF1
- new net N$40: U$2.PC13
- new net N$41: U$2.PB8
- new net N$42: U$2.BOOT0
- new net N$43: U$2.PB5
- new net N$44: U$2.PD2
- new net N$45: U$2.PC12
- new net N$46: U$2.PC11
- new net N$47: U$2.PC10
- new net N$48: U$2.PA15
- new net N$49: U$2.PA8
- new net N$50: U$2.PC9
- new net N$51: U$2.PC8
- new net N$52: U$2.PC7
- new net N$53: U$2.PC6
- new net N$54: U$2.PC14
- new net N$55: U$2.PC15
- new net N$56: U$2.VBAT
- new net N$57: U$2.PC0
- new net N$58: U$2.PC1
- new net N$59: U$2.PC2
- new net N$60: U$2.PC3
- new net N$61: U$2.PB10
- new net N$62: U$12.LED
- new net N$66: U$12.A0
- new net N$67: U$12.RESET
- new net OLED_SPI_MISO: U$2.PB14
- new net OLED_SPI_MOSI: U$12.SDA, U$2.PB15
- new net OLED_SPI_SCK: U$12.SCK, U$2.PB13
- new net PB0: U$2.PB0
- new net PB9: U$2.PB9
- net RFM69_RESET: now also U$2.PF4; no longer U$2.PB9
- net RMF69_INTERRUPT_DIO0: now also U$2.PC4; no longer U$2.PB0
- net VCC: now also U$12.CS
Changed lines of the file:
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@@
 </segment>
 <segment>
-<pinref part="U$2" gate="G$1" pin="PB9"/>
-<wire x1="15.24" y1="132.08" x2="15.24" y2="134.62" width="0.1524" layer="91"/>
-<label x="15.24" y="137.16" size="1.778" layer="95" rot="R90"/>
+<pinref part="U$2" gate="G$1" pin="PF4"/>
+<wire x1="12.7" y1="63.5" x2="12.7" y2="60.96" width="0.1524" layer="91"/>
+<label x="12.7" y="58.42" size="1.778" layer="95" rot="R270"/>
 </segment>
 </net>
@@
 </segment>
 <segment>
-<pinref part="U$2" gate="G$1" pin="PB0"/>
-<wire x1="33.02" y1="63.5" x2="33.02" y2="60.96" width="0.1524" layer="91"/>
-<label x="33.02" y="58.42" size="1.778" layer="95" rot="R270"/>
+<pinref part="U$2" gate="G$1" pin="PC4"/>
+<wire x1="27.94" y1="63.5" x2="27.94" y2="60.96" width="0.1524" layer="91"/>
+<label x="27.94" y="58.42" size="1.778" layer="95" rot="R270"/>
 </segment>
 </net>
@@
 <pinref part="U$2" gate="G$1" pin="PA0"/>
 <wire x1="-5.08" y1="83.82" x2="-7.62" y2="83.82" width="0.1524" layer="91"/>
+<label x="-10.16" y="83.82" size="1.778" layer="95" rot="R180"/>
 </segment>
 </net>
@@
 <pinref part="U$2" gate="G$1" pin="PA1"/>
 <wire x1="-5.08" y1="81.28" x2="-7.62" y2="81.28" width="0.1524" layer="91"/>
+<label x="-10.16" y="81.28" size="1.778" layer="95" rot="R180"/>
 </segment>
 </net>
@@
 <pinref part="U$2" gate="G$1" pin="PA2"/>
 <wire x1="-5.08" y1="78.74" x2="-7.62" y2="78.74" width="0.1524" layer="91"/>
+<label x="-10.16" y="78.74" size="1.778" layer="95" rot="R180"/>
 </segment>
 </net>
@@
 <pinref part="U$2" gate="G$1" pin="PA3"/>
 <wire x1="10.16" y1="63.5" x2="10.16" y2="60.96" width="0.1524" layer="91"/>
+<label x="10.16" y="58.42" size="1.778" layer="95" rot="R270"/>
 </segment>
 </net>
@@
 </segment>
 </net>
-<net name="N$38" class="0">
+<net name="OLED_SPI_NSS" class="0">
 <segment>
 <pinref part="U$2" gate="G$1" pin="PB12"/>
 <wire x1="63.5" y1="78.74" x2="66.04" y2="78.74" width="0.1524" layer="91"/>
+<label x="68.58" y="78.74" size="1.778" layer="95"/>
 </segment>
 </net>
@@
 <segment>
 <pinref part="U$12" gate="G$1" pin="VCC"/>
-<wire x1="27.94" y1="271.78" x2="-2.54" y2="271.78" width="0.1524" layer="91"/>
+<wire x1="27.94" y1="271.78" x2="17.78" y2="271.78" width="0.1524" layer="91"/>
 <pinref part="U$9" gate="G$1" pin="VCC"/>
+<wire x1="17.78" y1="271.78" x2="-2.54" y2="271.78" width="0.1524" layer="91"/>
 <wire x1="-2.54" y1="271.78" x2="-2.54" y2="274.32" width="0.1524" layer="91"/>
+<pinref part="U$12" gate="G$1" pin="CS"/>
+<wire x1="27.94" y1="261.62" x2="17.78" y2="261.62" width="0.1524" layer="91"/>
+<wire x1="17.78" y1="261.62" x2="17.78" y2="271.78" width="0.1524" layer="91"/>
+<junction x="17.78" y="271.78"/>
 </segment>
 <segment>
@@
 </segment>
 </net>
+<net name="PB0" class="0">
+<segment>
+<pinref part="U$2" gate="G$1" pin="PB0"/>
+<wire x1="33.02" y1="63.5" x2="33.02" y2="60.96" width="0.1524" layer="91"/>
+<label x="33.02" y="58.42" size="1.778" layer="95" rot="R270"/>
+</segment>
+</net>
+<net name="OLED_SPI_SCK" class="0">
+<segment>
+<pinref part="U$2" gate="G$1" pin="PB13"/>
+<wire x1="63.5" y1="81.28" x2="66.04" y2="81.28" width="0.1524" layer="91"/>
+<label x="68.58" y="81.28" size="1.778" layer="95"/>
+</segment>
+<segment>
+<pinref part="U$12" gate="G$1" pin="SCK"/>
+<wire x1="27.94" y1="241.3" x2="25.4" y2="241.3" width="0.1524" layer="91"/>
+<label x="22.86" y="241.3" size="1.778" layer="95" rot="R180"/>
+</segment>
+</net>
+<net name="OLED_SPI_MISO" class="0">
+<segment>
+<pinref part="U$2" gate="G$1" pin="PB14"/>
+<wire x1="63.5" y1="83.82" x2="66.04" y2="83.82" width="0.1524" layer="91"/>
+<label x="68.58" y="83.82" size="1.778" layer="95"/>
+</segment>
+</net>
+<net name="OLED_SPI_MOSI" class="0">
+<segment>
+<pinref part="U$2" gate="G$1" pin="PB15"/>
+<wire x1="63.5" y1="86.36" x2="66.04" y2="86.36" width="0.1524" layer="91"/>
+<label x="68.58" y="86.36" size="1.778" layer="95"/>
+</segment>
+<segment>
+<pinref part="U$12" gate="G$1" pin="SDA"/>
+<wire x1="27.94" y1="246.38" x2="25.4" y2="246.38" width="0.1524" layer="91"/>
+<label x="22.86" y="246.38" size="1.778" layer="95" rot="R180"/>
+</segment>
+</net>
+<net name="PB9" class="0">
+<segment>
+<pinref part="U$2" gate="G$1" pin="PB9"/>
+<wire x1="15.24" y1="132.08" x2="15.24" y2="134.62" width="0.1524" layer="91"/>
+<label x="15.24" y="137.16" size="1.778" layer="95" rot="R90"/>
+</segment>
+</net>
+<net name="N$38" class="0">
+<segment>
+<pinref part="U$2" gate="G$1" pin="PF0"/>
+<wire x1="-5.08" y1="106.68" x2="-7.62" y2="106.68" width="0.1524" layer="91"/>
+<label x="-10.16" y="106.68" size="1.778" layer="95" rot="R180"/>
+</segment>
+</net>
+<net name="N$39" class="0">
+<segment>
+<pinref part="U$2" gate="G$1" pin="PF1"/>
+<wire x1="-5.08" y1="104.14" x2="-7.62" y2="104.14" width="0.1524" layer="91"/>
+<label x="-10.16" y="104.14" size="1.778" layer="95" rot="R180"/>
+</segment>
+</net>
+<net name="N$40" class="0">
+<segment>
+<pinref part="U$2" gate="G$1" pin="PC13"/>
+<wire x1="-5.08" y1="114.3" x2="-7.62" y2="114.3" width="0.1524" layer="91"/>
+<label x="-10.16" y="114.3" size="1.778" layer="95" rot="R180"/>
+</segment>
+</net>
+<net name="N$41" class="0">
+<segment>
+<pinref part="U$2" gate="G$1" pin="PB8"/>
+<wire x1="17.78" y1="132.08" x2="17.78" y2="134.62" width="0.1524" layer="91"/>
+</segment>
+</net>
+<net name="N$42" class="0">
+<segment>
+<pinref part="U$2" gate="G$1" pin="BOOT0"/>
+<wire x1="20.32" y1="132.08" x2="20.32" y2="134.62" width="0.1524" layer="91"/>
+</segment>
+</net>
+<net name="N$43" class="0">
+<segment>
+<pinref part="U$2" gate="G$1" pin="PB5"/>
+<wire x1="27.94" y1="132.08" x2="27.94" y2="134.62" width="0.1524" layer="91"/>
+</segment>
+</net>
+<net name="N$44" class="0">
+<segment>
+<pinref part="U$2" gate="G$1" pin="PD2"/>
+<wire x1="35.56" y1="132.08" x2="35.56" y2="134.62" width="0.1524" layer="91"/>
+</segment>
+</net>
+<net name="N$45" class="0">
+<segment>
+<pinref part="U$2" gate="G$1" pin="PC12"/>
+<wire x1="38.1" y1="132.08" x2="38.1" y2="134.62" width="0.1524" layer="91"/>
+</segment>
+</net>
+<net name="N$46" class="0">
+<segment>
+<pinref part="U$2" gate="G$1" pin="PC11"/>
+<wire x1="40.64" y1="132.08" x2="40.64" y2="134.62" width="0.1524" layer="91"/>
+</segment>
+</net>
+<net name="N$47" class="0">
+<segment>
+<pinref part="U$2" gate="G$1" pin="PC10"/>
+<wire x1="43.18" y1="132.08" x2="43.18" y2="134.62" width="0.1524" layer="91"/>
+</segment>
+</net>
+<net name="N$48" class="0">
+<segment>
+<pinref part="U$2" gate="G$1" pin="PA15"/>
+<wire x1="45.72" y1="132.08" x2="45.72" y2="134.62" width="0.1524" layer="91"/>
+</segment>
+</net>
+<net name="N$49" class="0">
+<segment>
+<pinref part="U$2" gate="G$1" pin="PA8"/>
+<wire x1="63.5" y1="99.06" x2="66.04" y2="99.06" width="0.1524" layer="91"/>
+</segment>
+</net>
+<net name="N$50" class="0">
+<segment>
+<pinref part="U$2" gate="G$1" pin="PC9"/>
+<wire x1="63.5" y1="96.52" x2="66.04" y2="96.52" width="0.1524" layer="91"/>
+</segment>
+</net>
+<net name="N$51" class="0">
+<segment>
+<pinref part="U$2" gate="G$1" pin="PC8"/>
+<wire x1="63.5" y1="93.98" x2="66.04" y2="93.98" width="0.1524" layer="91"/>
+</segment>
+</net>
+<net name="N$52" class="0">
+<segment>
+<pinref part="U$2" gate="G$1" pin="PC7"/>
+<wire x1="63.5" y1="91.44" x2="66.04" y2="91.44" width="0.1524" layer="91"/>
+</segment>
+</net>
+<net name="N$53" class="0">
+<segment>
+<pinref part="U$2" gate="G$1" pin="PC6"/>
+<wire x1="63.5" y1="88.9" x2="66.04" y2="88.9" width="0.1524" layer="91"/>
+</segment>
+</net>
+<net name="N$54" class="0">
+<segment>
+<pinref part="U$2" gate="G$1" pin="PC14"/>
+<wire x1="-5.08" y1="111.76" x2="-7.62" y2="111.76" width="0.1524" layer="91"/>
+</segment>
+</net>
+<net name="N$55" class="0">
+<segment>
+<pinref part="U$2" gate="G$1" pin="PC15"/>
+<wire x1="-5.08" y1="109.22" x2="-7.62" y2="109.22" width="0.1524" layer="91"/>
+</segment>
+</net>
+<net name="N$56" class="0">
+<segment>
+<pinref part="U$2" gate="G$1" pin="VBAT"/>
+<wire x1="-5.08" y1="116.84" x2="-7.62" y2="116.84" width="0.1524" layer="91"/>
+</segment>
+</net>
+<net name="N$57" class="0">
+<segment>
+<pinref part="U$2" gate="G$1" pin="PC0"/>
+<wire x1="-5.08" y1="99.06" x2="-7.62" y2="99.06" width="0.1524" layer="91"/>
+</segment>
+</net>
+<net name="N$58" class="0">
+<segment>
+<pinref part="U$2" gate="G$1" pin="PC1"/>
+<wire x1="-5.08" y1="96.52" x2="-7.62" y2="96.52" width="0.1524" layer="91"/>
+</segment>
+</net>
+<net name="N$59" class="0">
+<segment>
+<pinref part="U$2" gate="G$1" pin="PC2"/>
+<wire x1="-5.08" y1="93.98" x2="-7.62" y2="93.98" width="0.1524" layer="91"/>
+</segment>
+</net>
+<net name="N$60" class="0">
+<segment>
+<pinref part="U$2" gate="G$1" pin="PC3"/>
+<wire x1="-5.08" y1="91.44" x2="-7.62" y2="91.44" width="0.1524" layer="91"/>
+</segment>
+</net>
+<net name="N$61" class="0">
+<segment>
+<pinref part="U$2" gate="G$1" pin="PB10"/>
+<wire x1="40.64" y1="63.5" x2="40.64" y2="60.96" width="0.1524" layer="91"/>
+</segment>
+</net>
+<net name="N$66" class="0">
+<segment>
+<pinref part="U$12" gate="G$1" pin="A0"/>
+<wire x1="27.94" y1="251.46" x2="25.4" y2="251.46" width="0.1524" layer="91"/>
+</segment>
+</net>
+<net name="N$67" class="0">
+<segment>
+<pinref part="U$12" gate="G$1" pin="RESET"/>
+<wire x1="27.94" y1="256.54" x2="25.4" y2="256.54" width="0.1524" layer="91"/>
+</segment>
+</net>
+<net name="N$62" class="0">
+<segment>
+<pinref part="U$12" gate="G$1" pin="LED"/>
+<wire x1="27.94" y1="236.22" x2="22.86" y2="236.22" width="0.1524" layer="91"/>
+</segment>
+</net>

Commit message: Updated design
Connections:
- net N$28 renamed TSC_G3_IO4
- net N$31 renamed SYS_JTMS_SWDIO
- net N$32 renamed SYS_JTCK-SWCLK
- net N$38 renamed RCC_OSC_IN
- net N$39 renamed RCC_OSC_OUT
- net N$40 renamed LED_STATUS
- net N$41 renamed TIM_IR_MAIN_SIGNAL
- net N$42 renamed BOOT0
- net PB9 renamed IR_OUT
- removed net N$22: U$2.PA0
- removed net N$23: U$2.PA1
- removed net N$24: U$2.PA2
- removed net N$25: U$2.PA3
- removed net N$26: U$2.PC5
- removed net N$27: U$2.PB1
- removed net N$33: U$2.PB3
- removed net N$34: U$2.PB4
- removed net N$35: U$2.PB6
- removed net N$36: U$2.PB7
- removed net PB0: U$2.PB0
- removed net TOUCH0: R20.1
- removed net TOUCH1: R11.1
- removed net TOUCH2: R12.1
- removed net TOUCH3: R13.1
- removed net TOUCH4: R14.1
- removed net TOUCH5: R15.1
- removed net TOUCH6: R16.1
- removed net TOUCH7: R17.1
- removed net TOUCH8: R18.1
- removed net TOUCH9: R19.1
- removed net TOUCHHOOK: R21.1
- new net TSC_G1_IO1: R17.1, U$2.PA0
- new net TSC_G1_IO2: R16.1, U$2.PA1
- new net TSC_G1_IO3: R15.1, U$2.PA2
- new net TSC_G1_IO4: R14.1, U$2.PA3
- new net TSC_G3_IO1: R13.1, U$2.PC5
- new net TSC_G3_IO2: R12.1, U$2.PB0
- new net TSC_G3_IO3: R11.1, U$2.PB1
- new net TSC_G5_IO1: R21.1, U$2.PB3
- new net TSC_G5_IO2: R20.1, U$2.PB4
- new net TSC_G5_IO3: R19.1, U$2.PB6
- new net TSC_G5_IO4: R18.1, U$2.PB7
