File: hardware/board/dc25-darknet-dialer-eaglev8.sch (EAGLE design)
At the start: 83 parts, among them SW1 RESET, X1 USB-MICROB, Y1 RESONATORSMD

Commit message: added stlink connector to lbr moved radio spi from spi1 to spi3 to free up pins for touch sensening
Parts:
- added LED13: (no value), SYNShop:LEDREVERSEMOUNT
- added R28: (no value), SYNShop:RESISTOR1206
- added STLINK: STLINK-V2-CONNECTOR, darknet_parts_library:STLINK-V2-CONNECTOR
Connections:
- net N$43 renamed TIM_IR_CARRIER_FREQ
- removed net N$44: U$2.PD2
- removed net N$45: U$2.PC12
- removed net N$46: U$2.PA10
- removed net N$48: U$2.PA9
- removed net N$61: U$2.PB11
- removed net N$66: U$12.A0
- removed net N$67: U$12.RESET
- removed net OLED_LED: U$12.LED, U$2.PC7
- removed net OLED_SPI_MISO: U$2.PB14
- new net N$29: LED13.A, R28.2
- new net N$50: U$2.PA7
- new net OLED_BACK_LIT: U$12.LED, U$2.PC6
- new net OLED_DATA_CMD: U$12.A0, U$2.PB14
- new net OLED_RESET: U$12.RESET, U$2.PC7
- new net RMF69_INTERRUPT_DIO1: U$15.DIO1, U$2.PB11
- new net TSC_G2_I01: R18.1, U$2.PA4
- new net TSC_G2_I02: R17.1, U$2.PA5
- new net TSC__G2_I03: U$2.PA6
- net GND: now also LED13.C, STLINK.GND
- net IR_RCV: now also U$2.PD2; no longer U$2.PC0
- net LED10: now also U$2.PA10; no longer U$2.PA15
- net LED8: now also U$2.PC0; no longer U$2.PC11
- net LED9: now also U$2.PA9; no longer U$2.PC10
- net LED_STATUS: now also R28.1
- net OLED_CS: no longer U$2.PC6
- net RFM69_SPI_MISO: now also U$2.PC11; no longer U$2.PA6
- net RFM69_SPI_MOSI: now also U$2.PC12; no longer U$2.PA7
- net RFM69_SPI_NSS: now also U$2.PA15; no longer U$2.PA4
- net RFM69_SPI_SCK: now also U$2.PC10; no longer U$2.PA5
- net RMF69_INTERRUPT_DIO0: now also U$15.DIO0; no longer U$15.DIO1
- net SYS_JTCK-SWCLK: now also STLINK.SWDCLK
- net SYS_JTMS_SWDIO: now also STLINK.SWDIO
- net TSC_G1_IO1: now also R16.1; no longer R17.1
- net TSC_G1_IO2: now also R15.1; no longer R16.1
- net TSC_G1_IO3: now also R14.1; no longer R15.1
- net TSC_G1_IO4: no longer R14.1
- net TSC_G5_IO4: no longer R18.1
- net VCC: now also STLINK.VCC
Other:
- note added: "I currently have the chip configured to use Hardware IR, hence the P57: TIM_IR_CARRIER_FREQ, we'll need to switch back to software or write for hw IR"

Commit message: updates to only have 1 pin for IR timer added todo list
Connections:
- removed net TIM_IR_MAIN_SIGNAL: LED12.C, U$2.PB8
- new net SD_CARD_CS: U$2.PB5
- net TIM_IR_CARRIER_FREQ: now also LED12.C, U$2.PB8; no longer U$2.PB5
Changed lines of the file:
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@@
 </segment>
 </net>
-<net name="TIM_IR_MAIN_SIGNAL" class="0">
+<net name="TSC_G5_IO4" class="0">
+<segment>
+<pinref part="U$2" gate="G$1" pin="PB7"/>
+<wire x1="22.86" y1="132.08" x2="22.86" y2="134.62" width="0.1524" layer="91"/>
+<label x="22.86" y="137.16" size="1.778" layer="95" rot="R90"/>
+</segment>
+</net>
+<net name="TIM_IR_CARRIER_FREQ" class="0">
+<segment>
+<pinref part="LED12" gate="G$1" pin="C"/>
+<wire x1="195.58" y1="208.28" x2="200.66" y2="208.28" width="0.1524" layer="91"/>
+<label x="203.2" y="208.28" size="1.778" layer="95"/>
+</segment>
 <segment>
 <pinref part="U$2" gate="G$1" pin="PB8"/>
 <wire x1="17.78" y1="132.08" x2="17.78" y2="134.62" width="0.1524" layer="91"/>
 <label x="17.78" y="137.16" size="1.778" layer="95" rot="R90"/>
-</segment>
-<segment>
-<pinref part="LED12" gate="G$1" pin="C"/>
-<wire x1="195.58" y1="208.28" x2="200.66" y2="208.28" width="0.1524" layer="91"/>
-<label x="203.2" y="208.28" size="1.778" layer="95"/>
-</segment>
-</net>
-<net name="TSC_G5_IO4" class="0">
-<segment>
-<pinref part="U$2" gate="G$1" pin="PB7"/>
-<wire x1="22.86" y1="132.08" x2="22.86" y2="134.62" width="0.1524" layer="91"/>
-<label x="22.86" y="137.16" size="1.778" layer="95" rot="R90"/>
-</segment>
-</net>
-<net name="TIM_IR_CARRIER_FREQ" class="0">
-<segment>
-<pinref part="U$2" gate="G$1" pin="PB5"/>
-<wire x1="27.94" y1="132.08" x2="27.94" y2="134.62" width="0.1524" layer="91"/>
-<label x="27.94" y="137.16" size="1.778" layer="95" rot="R90"/>
 </segment>
 </net>
@@
 </segment>
 </net>
+<net name="SD_CARD_CS" class="0">
+<segment>
+<pinref part="U$2" gate="G$1" pin="PB5"/>
+<wire x1="27.94" y1="132.08" x2="27.94" y2="134.62" width="0.1524" layer="91"/>
+<label x="27.94" y="137.16" size="1.778" layer="95" rot="R90"/>
+</segment>
+</net>

Commit message: added new part to library: SD_CARD_HEADER diff of todo.txt shows what else was completed on this check in. adding another doc on cap sense and updated stm32cube file
Parts:
- removed C1, C10, C11, C2, C3, C4, C5, C6, C7, C8, C9: (no value), SYNShop:C-USC0603
- added SAMPLE_CAP_G1, SAMPLE_CAP_G2, SAMPLE_CAP_G3, SAMPLE_CAP_G5: 10pF, SparkFun-Capacitors:10PF-50V-5%(0603)
- added SD_CARD_HEADER: SD_CARD_HEADER, darknet_parts_library:SD_CARD_HEADER
- R11, R12, R13, R14, R15, R16, R17, R18, R19, R20, R21: value (none) -> 1K
Connections:
- net OLED_BACK_LIT renamed LCD_BACK_LIT
- net OLED_DATA_CMD renamed LCD_DATA_CMD
- net OLED_RESET renamed LCD_RESET
- net OLED_SPI_MOSI renamed LCD_SPI_MOSI
- net OLED_SPI_SCK renamed LCD_SPI_SCK
- removed net OLED_CS: U$12.CS
- removed net OLED_SPI_NSS: U$2.PB12
- removed net SD_CARD_CS: U$2.PB5
- removed net TSC__G2_I03: U$2.PA6
- new net LCD_SPI_NSS: U$12.CS, U$2.PB12
- new net SD_CS: SD_CARD_HEADER.SD_CS, U$2.PB5
- new net TSC_G2_I03: SAMPLE_CAP_G2.1, U$2.PA6
- net GND: no longer C1.1, C10.1, C11.1, C2.1, C3.1, C4.1, C5.1, C6.1, C7.1, C8.1, C9.1
- net N$1: no longer C1.2
- net N$10: no longer C10.2
- net N$11: no longer C11.2
- net N$2: no longer C2.2
- net N$3: no longer C3.2
- net N$4: no longer C4.2
- net N$5: no longer C5.2
- net N$6: no longer C6.2
- net N$7: no longer C7.2
- net N$8: no longer C8.2
- net N$9: no longer C9.2
- net RFM69_SPI_MISO: now also SD_CARD_HEADER.SD_MISO
- net RFM69_SPI_MOSI: now also SD_CARD_HEADER.SD_MOSI
- net RFM69_SPI_SCK: now also SD_CARD_HEADER.SD_SCK
- net TSC_G1_IO4: now also SAMPLE_CAP_G1.1
- net TSC_G3_IO4: now also SAMPLE_CAP_G3.1
- net TSC_G5_IO4: now also SAMPLE_CAP_G5.1
Other:
- note removed: "I currently have the chip configured to use Hardware IR, hence the P57: TIM_IR_CARRIER_FREQ, we'll need to switch back to software or write for hw IR"
- moved on the sheet: R12, R13, R14, R15, R16, R17, R18, R19, R20, R21, TOUCH0, TOUCH2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

Commit message: Cleanup and update of schematic, added voltage regulator
Parts:
- added U$19: TLV702, darknet_parts_library:TLV702
- C12, C13, C14: value 100nF -> 0.1uF; device SYNShop:C-USC0603 -> darknet_parts_library:C-USC0603
- C15: value 10nF -> 0.01uF; device SYNShop:C-USC0603 -> darknet_parts_library:C-USC0603
- C16, C17, C18: device SYNShop:C-USC0603 -> darknet_parts_library:C-USC0603
- C19, C20: value (none) -> 47pF; device SYNShop:C-USC0603 -> darknet_parts_library:C-USC0603
- C21: value (none) -> 1uF; device SYNShop:C-USC0603 -> darknet_parts_library:C-USC0603
- R1, R10, R2, R28, R3, R4, R5, R6, R7, R8, R9: device SYNShop:RESISTOR1206 -> darknet_parts_library:RESISTOR1206
- R11, R12, R13, R14, R15, R16, R17, R18, R19, R20, R21, R22, R23: device SYNShop:R-US_R0603 -> darknet_parts_library:RESISTOR0603-RES
- R24: device SYNShop:R-US_0309/12 -> darknet_parts_library:R-US_0309/12
- R25: device SYNShop:R-US_0309/12 -> darknet_parts_library:RESISTOR0603-RES
- R26, R27: value (none) -> 27; device SYNShop:R-US_R0603 -> darknet_parts_library:RESISTOR0603-RES
- SAMPLE_CAP_G1, SAMPLE_CAP_G2, SAMPLE_CAP_G3, SAMPLE_CAP_G5: value 10pF -> 0.047uF; device SparkFun-Capacitors:10PF-50V-5%(0603) -> darknet_parts_library:C-USC0603
- X1: value USB-MICROB -> 10118193-0001LF
Connections:
- removed net N$31: F1.2
- new net N$30: F1.2, U$19.EN, U$19.VIN
- net GND: now also SAMPLE_CAP_G1.2, SAMPLE_CAP_G2.2, SAMPLE_CAP_G3.2, SAMPLE_CAP_G5.2, U$19.GND
- net USB_DM: now also R26.2
- net USB_DP: now also R27.2
- net VCC: now also U$19.VOUT
Other:
- note added: "Bypass Capacitors for STM32"
- moved on the sheet: C12, C13, C14, C15, C16, C17, C18, C19, C20, C21, CN1, F1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
