File: hardware/board/dc25-darknet-dialer-eaglev8.sch (EAGLE design)
At the start: 84 parts, among them SW1 RESET, X1 10118193-0001LF, Y1 RESONATORSMD

Commit message: Changed status LED for board debugging
Parts:
- LED13: device SYNShop:LEDREVERSEMOUNT -> SYNShop:LED0603
- R28: device darknet_parts_library:RESISTOR1206 -> darknet_parts_library:RESISTOR0603-RES
Changed lines of the file:
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@@
 <grid distance="0.1" unitdist="inch" unit="inch" style="lines" multiple="1" display="no" altdistance="0.01" altunitdist="inch" altunit="inch"/>
 <layers>
-<layer number="1" name="Top" color="4" fill="1" visible="no" active="no"/>
-<layer number="2" name="Route2" color="1" fill="3" visible="no" active="no"/>
-<layer number="3" name="Route3" color="4" fill="3" visible="no" active="no"/>
-<layer number="4" name="Route4" color="1" fill="4" visible="no" active="no"/>
-<layer number="5" name="Route5" color="4" fill="4" visible="no" active="no"/>
-<layer number="6" name="Route6" color="1" fill="8" visible="no" active="no"/>
-<layer number="7" name="Route7" color="4" fill="8" visible="no" active="no"/>
-<layer number="8" name="Route8" color="1" fill="2" visible="no" active="no"/>
-<layer number="9" name="Route9" color="4" fill="2" visible="no" active="no"/>
-<layer number="10" name="Route10" color="1" fill="7" visible="no" active="no"/>
-<layer number="11" name="Route11" color="4" fill="7" visible="no" active="no"/>
-<layer number="12" name="Route12" color="1" fill="5" visible="no" active="no"/>
-<layer number="13" name="Route13" color="4" fill="5" visible="no" active="no"/>
-<layer number="14" name="Route14" color="1" fill="6" visible="no" active="no"/>
-<layer number="15" name="Route15" color="4" fill="6" visible="no" active="no"/>
-<layer number="16" name="Bottom" color="1" fill="1" visible="no" active="no"/>
-<layer number="17" name="Pads" color="2" fill="1" visible="no" active="no"/>
-<layer number="18" name="Vias" color="2" fill="1" visible="no" active="no"/>
-<layer number="19" name="Unrouted" color="6" fill="1" visible="no" active="no"/>
-<layer number="20" name="Dimension" color="15" fill="1" visible="no" active="no"/>
-<layer number="21" name="tPlace" color="7" fill="1" visible="no" active="no"/>
-<layer number="22" name="bPlace" color="7" fill="1" visible="no" active="no"/>
-<layer number="23" name="tOrigins" color="15" fill="1" visible="no" active="no"/>
-<layer number="24" name="bOrigins" color="15" fill="1" visible="no" active="no"/>
-<layer number="25" name="tNames" color="7" fill="1" visible="no" active="no"/>
-<layer number="26" name="bNames" color="7" fill="1" visible="no" active="no"/>
-<layer number="27" name="tValues" color="7" fill="1" visible="no" active="no"/>
-<layer number="28" name="bValues" color="7" fill="1" visible="no" active="no"/>
+<layer number="1" name="Top" color="4" fill="1" visible="yes" active="no"/>
+<layer number="2" name="Route2" color="1" fill="3" visible="yes" active="no"/>
+<layer number="3" name="Route3" color="4" fill="3" visible="yes" active="no"/>
+<layer number="4" name="Route4" color="1" fill="4" visible="yes" active="no"/>
+<layer number="5" name="Route5" color="4" fill="4" visible="yes" active="no"/>
+<layer number="6" name="Route6" color="1" fill="8" visible="yes" active="no"/>
+<layer number="7" name="Route7" color="4" fill="8" visible="yes" active="no"/>
+<layer number="8" name="Route8" color="1" fill="2" visible="yes" active="no"/>
+<layer number="9" name="Route9" color="4" fill="2" visible="yes" active="no"/>
+<layer number="10" name="Route10" color="1" fill="7" visible="yes" active="no"/>
+<layer number="11" name="Route11" color="4" fill="7" visible="yes" active="no"/>
+<layer number="12" name="Route12" color="1" fill="5" visible="yes" active="no"/>
+<layer number="13" name="Route13" color="4" fill="5" visible="yes" active="no"/>
+<layer number="14" name="Route14" color="1" fill="6" visible="yes" active="no"/>
+<layer number="15" name="Route15" color="4" fill="6" visible="yes" active="no"/>
+<layer number="16" name="Bottom" color="1" fill="1" visible="yes" active="no"/>
+<layer number="17" name="Pads" color="2" fill="1" visible="yes" active="no"/>
+<layer number="18" name="Vias" color="2" fill="1" visible="yes" active="no"/>
+<layer number="19" name="Unrouted" color="6" fill="1" visible="yes" active="no"/>
+<layer number="20" name="Dimension" color="15" fill="1" visible="yes" active="no"/>
+<layer number="21" name="tPlace" color="7" fill="1" visible="yes" active="no"/>
+<layer number="22" name="bPlace" color="7" fill="1" visible="yes" active="no"/>
+<layer number="23" name="tOrigins" color="15" fill="1" visible="yes" active="no"/>
+<layer number="24" name="bOrigins" color="15" fill="1" visible="yes" active="no"/>
+<layer number="25" name="tNames" color="7" fill="1" visible="yes" active="no"/>
+<layer number="26" name="bNames" color="7" fill="1" visible="yes" active="no"/>
+<layer number="27" name="tValues" color="7" fill="1" visible="yes" active="no"/>
+<layer number="28" name="bValues" color="7" fill="1" visible="yes" active="no"/>
 <layer number="29" name="tStop" color="7" fill="3" visible="no" active="no"/>
 <layer number="30" name="bStop" color="7" fill="6" visible="no" active="no"/>
@@
 <layer number="35" name="tGlue" color="7" fill="4" visible="no" active="no"/>
 <layer number="36" name="bGlue" color="7" fill="5" visible="no" active="no"/>
-<layer number="37" name="tTest" color="7" fill="1" visible="no" active="no"/>
-<layer number="38" name="bTest" color="7" fill="1" visible="no" active="no"/>
+<layer number="37" name="tTest" color="7" fill="1" visible="yes" active="no"/>
+<layer number="38" name="bTest" color="7" fill="1" visible="yes" active="no"/>
 <layer number="39" name="tKeepout" color="4" fill="11" visible="no" active="no"/>
 <layer number="40" name="bKeepout" color="1" fill="11" visible="no" active="no"/>
@@
 <layer number="44" name="Drills" color="7" fill="1" visible="no" active="no"/>
 <layer number="45" name="Holes" color="7" fill="1" visible="no" active="no"/>
-<layer number="46" name="Milling" color="3" fill="1" visible="no" active="no"/>
-<layer number="47" name="Measures" color="7" fill="1" visible="no" active="no"/>
-<layer number="48" name="Document" color="7" fill="1" visible="no" active="no"/>
-<layer number="49" name="Reference" color="7" fill="1" visible="no" active="no"/>
-<layer number="50" name="dxf" color="7" fill="1" visible="no" active="no"/>
-<layer number="51" name="tDocu" color="7" fill="1" visible="no" active="no"/>
-<layer number="52" name="bDocu" color="7" fill="1" visible="no" active="no"/>
-<layer number="53" name="tGND_GNDA" color="7" fill="9" visible="no" active="no"/>
-<layer number="54" name="bGND_GNDA" color="1" fill="9" visible="no" active="no"/>
-<layer number="56" name="wert" color="7" fill="1" visible="no" active="no"/>
-<layer number="57" name="tCAD" color="7" fill="1" visible="no" active="no"/>
-<layer number="59" name="tCarbon" color="7" fill="1" visible="no" active="no"/>
-<layer number="60" name="bCarbon" color="7" fill="1" visible="no" active="no"/>
+<layer number="46" name="Milling" color="3" fill="1" visible="yes" active="no"/>
+<layer number="47" name="Measures" color="7" fill="1" visible="yes" active="no"/>
+<layer number="48" name="Document" color="7" fill="1" visible="yes" active="no"/>
+<layer number="49" name="Reference" color="7" fill="1" visible="yes" active="no"/>
+<layer number="50" name="dxf" color="7" fill="1" visible="yes" active="no"/>
+<layer number="51" name="tDocu" color="7" fill="1" visible="yes" active="no"/>
+<layer number="52" name="bDocu" color="7" fill="1" visible="yes" active="no"/>
+<layer number="53" name="tGND_GNDA" color="7" fill="9" visible="yes" active="no"/>
+<layer number="54" name="bGND_GNDA" color="1" fill="9" visible="yes" active="no"/>
+<layer number="56" name="wert" color="7" fill="1" visible="yes" active="no"/>
+<layer number="57" name="tCAD" color="7" fill="1" visible="yes" active="no"/>
+<layer number="59" name="tCarbon" color="7" fill="1" visible="yes" active="no"/>
+<layer number="60" name="bCarbon" color="7" fill="1" visible="yes" active="no"/>
 <layer number="90" name="Modules" color="5" fill="1" visible="yes" active="yes"/>
 <layer number="91" name="Nets" color="2" fill="1" visible="yes" active="yes"/>
@@
 <part name="C21" library="darknet_parts_library" deviceset="C-US" device="C0603" value="1uF"/>
 <part name="U$13" library="SYNShop" deviceset="VCC" device=""/>
-<part name="LED13" library="SYNShop" deviceset="LED" device="REVERSEMOUNT"/>
-<part name="R28" library="darknet_parts_library" deviceset="RESISTOR" device="1206"/>
+<part name="LED13" library="SYNShop" deviceset="LED" device="0603"/>
+<part name="R28" library="darknet_parts_library" deviceset="RESISTOR" device="0603-RES"/>
 <part name="STLINK" library="darknet_parts_library" deviceset="STLINK-V2-CONNECTOR" device=""/>
 <part name="SAMPLE_CAP_G3" library="darknet_parts_library" deviceset="C-US" device="C0603" value="0.047uF"/>

Commit message: Finished routing
Parts:
- added U$12: KRUX_LOGO, darknet_parts_library:KRUX_LOGO
- added U$23: CMD_C0DE_LOGO, darknet_parts_library:CMD_C0DE_LOGO
- R24: device darknet_parts_library:R-US_0309/12 -> darknet_parts_library:R-US_0207/7
- U$17: device SYNShop:SOP22 -> darknet_parts_library:SOP22
Connections:
- net TSC_G2_I03 renamed TSC_G2_IO3
- removed net TSC_G2_I01: R18.1, U$2.PA4
- removed net TSC_G2_I02: R17.1, U$2.PA5
- new net TSC_G2_IO1: R14.1, U$2.PA4
- new net TSC_G2_IO2: R15.1, U$2.PA5
- net GND: now also CN1.1; no longer CN1.2
- net TSC_G1_IO1: now also R18.1; no longer R16.1
- net TSC_G1_IO2: now also R17.1; no longer R15.1
- net TSC_G1_IO3: now also R16.1; no longer R14.1
- net VCC1: now also CN1.2; no longer CN1.1
Other:
- note removed: "Note need to check on power connection / battery"
- moved on the sheet: CN1, STLINK
Changed lines of the file:
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@@
 <part name="X1" library="SYNShop" deviceset="USB" device="-MICROB" value="10118193-0001LF"/>
 <part name="U$16" library="SYNShop" deviceset="VCC0" device="" value="5V"/>
-<part name="U$17" library="SYNShop" deviceset="SOP22" device=""/>
+<part name="U$17" library="darknet_parts_library" deviceset="SOP22" device=""/>
 <part name="LED12" library="SYNShop" deviceset="LED" device="5MM"/>
-<part name="R24" library="darknet_parts_library" deviceset="R-US_" device="0309/12"/>
+<part name="R24" library="darknet_parts_library" deviceset="R-US_" device="0207/7"/>
 <part name="GND27" library="SYNShop" deviceset="GND" device=""/>
 <part name="U$18" library="SYNShop" deviceset="VCC" device=""/>
@@
 <part name="L3" library="darknet_parts_library" deviceset="INDUCTOR" device="0603" value="4.7nH"/>
 <part name="U$22" library="darknet_parts_library" deviceset="ST7735S_LCD_MODULE" device=""/>
+<part name="U$12" library="darknet_parts_library" deviceset="KRUX_LOGO" device=""/>
+<part name="U$23" library="darknet_parts_library" deviceset="CMD_C0DE_LOGO" device=""/>
 </parts>
 <sheets>
 <sheet>
 <plain>
-<text x="162.56" y="289.56" size="1.778" layer="91">Note need to check on power connection / battery</text>
 <text x="83.82" y="406.4" size="1.778" layer="91">3.3V LDO Voltage regulator
 Here.. need to make part</text>
@@
 <instance part="GND27" gate="1" x="264.16" y="220.98"/>
 <instance part="U$18" gate="G$1" x="264.16" y="241.3"/>
-<instance part="CN1" gate="G$1" x="167.64" y="302.26"/>
+<instance part="CN1" gate="G$1" x="160.02" y="304.8" rot="R180"/>
 <instance part="SW1" gate="G$1" x="236.22" y="347.98"/>
 <instance part="R25" gate="G$1" x="236.22" y="363.22" rot="R90"/>
@@
 <instance part="LED13" gate="G$1" x="254" y="76.2" rot="R90"/>
 <instance part="R28" gate="G$1" x="246.38" y="76.2"/>
-<instance part="STLINK" gate="G$1" x="256.54" y="266.7"/>
+<instance part="STLINK" gate="G$1" x="238.76" y="274.32"/>
 <instance part="SAMPLE_CAP_G3" gate="G$1" x="332.74" y="187.96" rot="R90"/>
 <instance part="SAMPLE_CAP_G1" gate="G$1" x="332.74" y="144.78" rot="R90"/>
@@
 <instance part="GND13" gate="1" x="340.36" y="182.88"/>
 <instance part="U$14" gate="G$1" x="264.16" y="274.32"/>
-<instance part="GND14" gate="1" x="264.16" y="259.08"/>
+<instance part="GND14" gate="1" x="264.16" y="256.54"/>
 <instance part="U$19" gate="G$1" x="101.6" y="391.16"/>
 <instance part="GND15" gate="1" x="101.6" y="373.38"/>
@@
 <instance part="L3" gate="G$1" x="137.16" y="157.48" rot="R180"/>
 <instance part="U$22" gate="G$1" x="116.84" y="241.3"/>
+<instance part="U$12" gate="G$1" x="22.86" y="5.08"/>
+<instance part="U$23" gate="G$1" x="33.02" y="5.08"/>
 </instances>
 <busses>
@@
 </segment>
 <segment>
-<pinref part="CN1" gate="G$1" pin="2"/>
 <pinref part="GND24" gate="1" pin="GND"/>
-<wire x1="165.1" y1="302.26" x2="142.24" y2="302.26" width="0.1524" layer="91"/>
 <wire x1="142.24" y1="302.26" x2="142.24" y2="294.64" width="0.1524" layer="91"/>
+<wire x1="142.24" y1="302.26" x2="162.56" y2="302.26" width="0.1524" layer="91"/>
+<pinref part="CN1" gate="G$1" pin="1"/>
 </segment>
 <segment>
@@
 <segment>
 <pinref part="STLINK" gate="G$1" pin="GND"/>
-<wire x1="243.84" y1="264.16" x2="264.16" y2="264.16" width="0.1524" layer="91"/>
-<wire x1="264.16" y1="264.16" x2="264.16" y2="261.62" width="0.1524" layer="91"/>
+<wire x1="248.92" y1="264.16" x2="264.16" y2="264.16" width="0.1524" layer="91"/>
+<wire x1="264.16" y1="264.16" x2="264.16" y2="259.08" width="0.1524" layer="91"/>
 <pinref part="GND14" gate="1" pin="GND"/>
 </segment>
@@
 </segment>
 <segment>
+<pinref part="R18" gate="G$1" pin="1"/>
+<wire x1="302.26" y1="96.52" x2="297.18" y2="96.52" width="0.1524" layer="91"/>
+<label x="294.64" y="96.52" size="1.778" layer="95" rot="R180"/>
+</segment>
+</net>
+<net name="TSC_G1_IO2" class="0">
+<segment>
+<pinref part="U$2" gate="G$1" pin="PA1"/>
+<wire x1="58.42" y1="68.58" x2="55.88" y2="68.58" width="0.1524" layer="91"/>
+<label x="53.34" y="68.58" size="1.778" layer="95" rot="R180"/>
+</segment>
+<segment>
+<pinref part="R17" gate="G$1" pin="1"/>
+<wire x1="302.26" y1="106.68" x2="297.18" y2="106.68" width="0.1524" layer="91"/>
+<label x="294.64" y="106.68" size="1.778" layer="95" rot="R180"/>
+</segment>
+</net>
+<net name="TSC_G1_IO3" class="0">
+<segment>
+<pinref part="U$2" gate="G$1" pin="PA2"/>
+<wire x1="58.42" y1="66.04" x2="55.88" y2="66.04" width="0.1524" layer="91"/>
+<label x="53.34" y="66.04" size="1.778" layer="95" rot="R180"/>
+</segment>
+<segment>
 <pinref part="R16" gate="G$1" pin="1"/>
 <wire x1="302.26" y1="121.92" x2="297.18" y2="121.92" width="0.1524" layer="91"/>
@@
 </segment>
 </net>
-<net name="TSC_G1_IO2" class="0">
-<segment>
-<pinref part="U$2" gate="G$1" pin="PA1"/>
-<wire x1="58.42" y1="68.58" x2="55.88" y2="68.58" width="0.1524" layer="91"/>
-<label x="53.34" y="68.58" size="1.778" layer="95" rot="R180"/>
-</segment>
-<segment>
-<pinref part="R15" gate="G$1" pin="1"/>
-<wire x1="302.26" y1="129.54" x2="297.18" y2="129.54" width="0.1524" layer="91"/>
-<label x="294.64" y="129.54" size="1.778" layer="95" rot="R180"/>
-</segment>
-</net>
-<net name="TSC_G1_IO3" class="0">
-<segment>
-<pinref part="U$2" gate="G$1" pin="PA2"/>
-<wire x1="58.42" y1="66.04" x2="55.88" y2="66.04" width="0.1524" layer="91"/>
-<label x="53.34" y="66.04" size="1.778" layer="95" rot="R180"/>
-</segment>
-<segment>
-<pinref part="R14" gate="G$1" pin="1"/>
-<wire x1="302.26" y1="137.16" x2="297.18" y2="137.16" width="0.1524" layer="91"/>
-<label x="294.64" y="137.16" size="1.778" layer="95" rot="R180"/>
-</segment>
-</net>
 <net name="TSC_G1_IO4" class="0">
 <segment>
@@
 <segment>
 <pinref part="STLINK" gate="G$1" pin="SWDIO"/>
-<wire x1="243.84" y1="269.24" x2="266.7" y2="269.24" width="0.1524" layer="91"/>
+<wire x1="248.92" y1="269.24" x2="266.7" y2="269.24" width="0.1524" layer="91"/>
 <label x="269.24" y="269.24" size="1.778" layer="95"/>
 </segment>
@@
 <segment>
 <pinref part="STLINK" gate="G$1" pin="SWDCLK"/>
-<wire x1="243.84" y1="266.7" x2="266.7" y2="266.7" width="0.1524" layer="91"/>
+<wire x1="248.92" y1="266.7" x2="266.7" y2="266.7" width="0.1524" layer="91"/>
 <label x="269.24" y="266.7" size="1.778" layer="95"/>
 </segment>
@@
 <pinref part="STLINK" gate="G$1" pin="VCC"/>
 <pinref part="U$14" gate="G$1" pin="VCC"/>
-<wire x1="243.84" y1="271.78" x2="264.16" y2="271.78" width="0.1524" layer="91"/>
+<wire x1="248.92" y1="271.78" x2="264.16" y2="271.78" width="0.1524" layer="91"/>
 <wire x1="264.16" y1="271.78" x2="264.16" y2="274.32" width="0.1524" layer="91"/>
 </segment>
@@
 <pinref part="5V" gate="VCC0" pin="VCC0"/>
 <wire x1="60.96" y1="304.8" x2="60.96" y2="309.88" width="0.1524" layer="91"/>
+<junction x="86.36" y="304.8"/>
 </segment>
 <segment>
@@
 <junction x="129.54" y="304.8"/>
 <wire x1="142.24" y1="304.8" x2="142.24" y2="309.88" width="0.1524" layer="91"/>
-<pinref part="CN1" gate="G$1" pin="1"/>
-<wire x1="142.24" y1="304.8" x2="165.1" y2="304.8" width="0.1524" layer="91"/>
 <pinref part="3.7V" gate="G$1" pin="VCC1"/>
-<junction x="142.24" y="304.8"/>
+<wire x1="142.24" y1="304.8" x2="162.56" y2="304.8" width="0.1524" layer="91"/>
+<pinref part="CN1" gate="G$1" pin="2"/>
 </segment>
 <segment>
@@
 </segment>
 </net>
-<net name="TSC_G2_I01" class="0">
+<net name="TSC_G2_IO1" class="0">
 <segment>
 <pinref part="U$2" gate="G$1" pin="PA4"/>
@@
 </segment>
 <segment>
-<pinref part="R18" gate="G$1" pin="1"/>
-<wire x1="302.26" y1="96.52" x2="297.18" y2="96.52" width="0.1524" layer="91"/>
-<label x="294.64" y="96.52" size="1.778" layer="95" rot="R180"/>
-</segment>
-</net>
-<net name="TSC_G2_I02" class="0">
+<pinref part="R14" gate="G$1" pin="1"/>
+<wire x1="302.26" y1="137.16" x2="297.18" y2="137.16" width="0.1524" layer="91"/>
+<label x="294.64" y="137.16" size="1.778" layer="95" rot="R180"/>
+</segment>
+</net>
+<net name="TSC_G2_IO2" class="0">
 <segment>
 <pinref part="U$2" gate="G$1" pin="PA5"/>
@@
 </segment>
 <segment>
-<pinref part="R17" gate="G$1" pin="1"/>
-<wire x1="302.26" y1="106.68" x2="297.18" y2="106.68" width="0.1524" layer="91"/>
-<label x="294.64" y="106.68" size="1.778" layer="95" rot="R180"/>
-</segment>
-</net>
-<net name="TSC_G2_I03" class="0">
+<pinref part="R15" gate="G$1" pin="1"/>
+<wire x1="302.26" y1="129.54" x2="297.18" y2="129.54" width="0.1524" layer="91"/>
+<label x="294.64" y="129.54" size="1.778" layer="95" rot="R180"/>
+</segment>
+</net>
+<net name="TSC_G2_IO3" class="0">
 <segment>
 <pinref part="U$2" gate="G$1" pin="PA6"/>
