File: hardware/board/dc25-darknet-dialer-eaglev8.1.brd (EAGLE design)
At the start: 101.6 x 101.6 mm, 94 parts, among them J1 MF-CON-MICROUSB-RIGHT, SW1 RESET, U1 BU33SD5WG-TR, U2 MCP73831T-5ACI/OT, U3 SOP22FLAT, Y1 CSTCE8M00G52-R0

Commit message: Added audio out pads
Parts:
- removed R29: 2K DNP, darknet_parts_library:0603-RES
- added JP1, JP2: (no value), adafruit:1X01-CLEANBIG
- added R35: 2K DNP, darknet_parts_library:0603-RES
- R30: value 1K DNP -> 2K DNP
- R31: value 2K DNP -> 1K DNP
- moved R34 5.38 mm to (48.1, 33.6)
- moved R33 4.29 mm to (48.1, 35.7)
- moved R31 3.90 mm to (44.8, 35.7), turned to 180 degrees
- moved R30 2.14 mm to (44.8, 37.9), turned to 0 degrees
Connections:
- net AUDIO_1: now also R35.1; no longer R33.1
- net AUDIO_2: now also R34.1; no longer R31.1
- net AUDIO_3: now also R33.1; no longer R29.1
- net AUDIO_OUT: now also JP1.1
- net GND: now also JP2.1, R30.2; no longer R34.2
- net N$33: now also R35.2; no longer R33.2
- net N$34: now also R31.1, R34.2; no longer R30.1, R31.2
- net N$35: now also R30.1, R31.2, R33.2; no longer R29.2, R30.2, R34.1
Routing:
- net AUDIO_OUT: track 0.00 -> 2.41 mm
Changed lines of the file:
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@@
 <setting verticaltext="up"/>
 </settings>
-<grid distance="0.003125" unitdist="inch" unit="inch" style="lines" multiple="1" display="yes" altdistance="0.025" altunitdist="inch" altunit="inch"/>
+<grid distance="0.0125" unitdist="inch" unit="inch" style="lines" multiple="1" display="yes" altdistance="0.025" altunitdist="inch" altunit="inch"/>
 <layers>
 <layer number="1" name="Top" color="4" fill="1" visible="yes" active="yes"/>
@@
 </element>
 <element name="R2" library="darknet_parts_library" package="1206" value="CRCW120647R0JNEA" x="69.215" y="82.07375" smashed="yes" rot="MR90">
-<attribute name="NAME" x="70.6755" y="81.5975" size="0.6096" layer="26" font="vector" rot="MR90"/>
+<attribute name="NAME" x="67.183" y="81.5975" size="0.6096" layer="26" font="vector" rot="MR90"/>
 </element>
 <element name="R3" library="darknet_parts_library" package="1206" value="CRCW120647R0JNEA" x="47.069375" y="80.16875" smashed="yes" rot="MR0">
@@
 </element>
 <element name="R12" library="darknet_parts_library" package="0603-RES" value="1K" x="59.3725" y="79.53375" smashed="yes" rot="MR180">
-<attribute name="NAME" x="56.642" y="78.724125" size="0.6096" layer="26" font="vector" rot="MR90"/>
+<attribute name="NAME" x="57.165875" y="79.1845" size="0.6096" layer="26" font="vector" rot="MR0"/>
 </element>
 <element name="R13" library="darknet_parts_library" package="0603-RES" value="1K" x="41.75125" y="79.53375" smashed="yes" rot="MR0">
@@
 </element>
 <element name="R19" library="darknet_parts_library" package="0603-RES" value="1K" x="59.293125" y="23.97125" smashed="yes" rot="MR180">
-<attribute name="NAME" x="58.404125" y="25.669875" size="0.6096" layer="26" font="vector" rot="MR180"/>
+<attribute name="NAME" x="58.404125" y="23.129875" size="0.6096" layer="26" font="vector" rot="MR180"/>
 </element>
 <element name="R20" library="darknet_parts_library" package="0603-RES" value="1K" x="75.803125" y="32.86125" smashed="yes" rot="MR180">
@@
 </element>
 <element name="U$11" library="darknet_parts_library" package="SPDT_SSAJ120100" value="SWITCH_SPDT" x="50.879375" y="84.93125" rot="MR270"/>
-<element name="R29" library="darknet_parts_library" package="0603-RES" value="2K DNP" x="48.10125" y="35.71875" smashed="yes" rot="MR0">
+<element name="R33" library="darknet_parts_library" package="0603-RES" value="2K DNP" x="48.10125" y="35.71875" smashed="yes" rot="MR0">
 <attribute name="NAME" x="49.990375" y="36.068" size="0.6096" layer="26" font="vector" rot="MR180"/>
 </element>
-<element name="R30" library="darknet_parts_library" package="0603-RES" value="1K DNP" x="44.846875" y="35.71875" smashed="yes" rot="MR180">
+<element name="R31" library="darknet_parts_library" package="0603-RES" value="1K DNP" x="44.846875" y="35.71875" smashed="yes" rot="MR180">
 <attribute name="NAME" x="43.037125" y="35.448875" size="0.6096" layer="26" font="vector" rot="MR0"/>
 </element>
-<element name="R31" library="darknet_parts_library" package="0603-RES" value="2K DNP" x="48.10125" y="33.575625" smashed="yes" rot="MR0">
+<element name="R34" library="darknet_parts_library" package="0603-RES" value="2K DNP" x="48.10125" y="33.575625" smashed="yes" rot="MR0">
 <attribute name="NAME" x="49.990375" y="33.8455" size="0.6096" layer="26" font="vector" rot="MR180"/>
 </element>
@@
 <attribute name="NAME" x="43.037125" y="33.226375" size="0.6096" layer="26" font="vector" rot="MR0"/>
 </element>
-<element name="R33" library="darknet_parts_library" package="0603-RES" value="2K DNP" x="48.10125" y="31.4325" smashed="yes" rot="MR0">
+<element name="R35" library="darknet_parts_library" package="0603-RES" value="2K DNP" x="48.10125" y="31.4325" smashed="yes" rot="MR0">
 <attribute name="NAME" x="49.990375" y="32.5755" size="0.6096" layer="26" font="vector" rot="MR180"/>
 </element>
@@
 <attribute name="NAME" x="42.95775" y="31.162625" size="0.6096" layer="26" rot="MR0"/>
 </element>
-<element name="R34" library="darknet_parts_library" package="0603-RES" value="2K DNP" x="44.846875" y="37.861875" smashed="yes" rot="MR0">
+<element name="R30" library="darknet_parts_library" package="0603-RES" value="2K DNP" x="44.846875" y="37.861875" smashed="yes" rot="MR0">
 <attribute name="NAME" x="43.037125" y="37.592" size="0.6096" layer="26" font="vector" rot="MR0"/>
+</element>
+<element name="JP1" library="adafruit" package="1X01-CLEANBIG" value="" x="44.45" y="29.21" smashed="yes">
+<attribute name="VALUE" x="43.18" y="26.035" size="1.27" layer="27"/>
+</element>
+<element name="JP2" library="adafruit" package="1X01-CLEANBIG" value="" x="46.99" y="29.21" smashed="yes">
+<attribute name="VALUE" x="45.72" y="26.035" size="1.27" layer="27"/>
 </element>
 </elements>
@@
 <contactref element="J1" pad="S4"/>
 <contactref element="J1" pad="S6"/>
-<contactref element="R34" pad="2"/>
+<contactref element="R30" pad="2"/>
 <wire x1="56.9125" y1="47.705" x2="56.27625" y2="47.705" width="0.3048" layer="16"/>
 <wire x1="56.27625" y1="47.705" x2="55.88" y2="48.10125" width="0.3048" layer="16"/>
@@
 <wire x1="54.13375" y1="48.10125" x2="54.85875" y2="48.10125" width="0.3048" layer="16"/>
 <wire x1="54.85875" y1="48.10125" x2="54.8625" y2="48.105" width="0.3048" layer="16"/>
+<contactref element="JP2" pad="1"/>
 <wire x1="95.063721875" y1="72.642596875" x2="94.17169375" y2="74.54373125" width="0" layer="19" extent="16-16"/>
 <wire x1="96.960971875" y1="68.562096875" x2="96.07800625" y2="70.46745625" width="0" layer="19" extent="16-16"/>
@@
 <signal name="AUDIO_1">
 <contactref element="U$2" pad="P41"/>
-<contactref element="R33" pad="1"/>
+<contactref element="R35" pad="1"/>
 <wire x1="54.8625" y1="51.105" x2="54.066875" y2="51.105" width="0.3048" layer="16"/>
 <wire x1="54.066875" y1="51.105" x2="53.895625" y2="51.27625" width="0.3048" layer="16"/>
@@
 <signal name="AUDIO_3">
 <contactref element="U$2" pad="P4"/>
-<contactref element="R29" pad="1"/>
+<contactref element="R33" pad="1"/>
 <wire x1="43.5625" y1="49.105" x2="44.319375" y2="49.105" width="0.3048" layer="16"/>
 <wire x1="44.319375" y1="49.105" x2="44.45" y2="48.974375" width="0.3048" layer="16"/>
@@
 <signal name="AUDIO_2">
 <contactref element="U$2" pad="P23"/>
-<contactref element="R31" pad="1"/>
+<contactref element="R34" pad="1"/>
 <wire x1="48.4625" y1="57.005" x2="48.4625" y2="51.70875" width="0.3048" layer="16"/>
 <wire x1="48.4625" y1="51.70875" x2="48.815625" y2="51.355625" width="0.3048" layer="16"/>
@@
 </signal>
 <signal name="N$33">
-<contactref element="R33" pad="2"/>
+<contactref element="R35" pad="2"/>
 <contactref element="C2" pad="1"/>
 <contactref element="R32" pad="1"/>
@@
 <signal name="N$34">
 <contactref element="R32" pad="2"/>
-<contactref element="R30" pad="1"/>
-<contactref element="R31" pad="2"/>
+<contactref element="R31" pad="1"/>
+<contactref element="R34" pad="2"/>
 <wire x1="43.996875" y1="35.71875" x2="43.996875" y2="33.995625" width="0.3048" layer="16"/>
 <wire x1="43.996875" y1="33.575625" x2="43.996875" y2="33.995625" width="0.3048" layer="16"/>
@@
 </signal>
 <signal name="N$35">
-<contactref element="R30" pad="2"/>
-<contactref element="R29" pad="2"/>
-<contactref element="R34" pad="1"/>
+<contactref element="R31" pad="2"/>
+<contactref element="R33" pad="2"/>
+<contactref element="R30" pad="1"/>
 <wire x1="47.25125" y1="35.71875" x2="45.696875" y2="35.71875" width="0.3048" layer="16"/>
 <wire x1="45.696875" y1="35.71875" x2="45.696875" y2="37.861875" width="0.3048" layer="16"/>
@@
 <signal name="AUDIO_OUT">
 <contactref element="C2" pad="2"/>
+<contactref element="JP1" pad="1"/>
+<wire x1="43.996875" y1="31.4325" x2="43.996875" y2="29.663125" width="0.3048" layer="16"/>
+<wire x1="43.996875" y1="29.663125" x2="44.45" y2="29.21" width="0.3048" layer="16"/>
 </signal>
 </signals>

Commit message: Updated switch hook, and removed solder paste for kit parts
Parts:
- LED1, LED10, LED2, LED3, LED4, LED5, LED6, LED7, LED8, LED9: device SYNShop:GULLWING_LED -> darknet_parts_library:GULLWING_LED_NOPASTE
- U$15: value RFM69HCWRFN69HCWSMD -> RFM69HCWRFM69HCWSMDNOPASTE; device SYNShop:16PIN-PCB-SMD -> SYNShop:16PIN-PCB-SMD-NOPASTE
- moved R18 1.27 mm to (42.1, 23.3)
- moved C25 0.83 mm to (48.0, 41.4), turned to 0 degrees
- moved R20 0.64 mm to (76.4, 32.9)
- moved R19 0.64 mm to (59.3, 23.3)
- moved LED8 0.16 mm to (38.4, 11.7)
Routing:
- net TSC_G5_IO2: track 31.6 -> 35.1 mm
- net TSC_G5_IO3: track 25.9 -> 29.3 mm
- net TSC_G5_IO1: track 30.2 -> 28.2 mm
- net N$8: track 4.96 -> 3.69 mm
- net TSC_G1_IO1: track 63.1 -> 64.3 mm
- net N$9: track 4.43 -> 3.76 mm
- net N$10: track 4.25 -> 3.66 mm
