File: hardware/board/dc25-darknet-dialer-eaglev8.2.brd (EAGLE design)
At the start: 101.6 x 101.6 mm, 96 parts, among them J1 MF-CON-MICROUSB-RIGHT, SW1 RESET, U1 BU33SD5WG-TR, U2 MCP73831T-5ACI/OT, U3 SOP22FLAT, Y1 CSTCE8M00G52-R0

Commit message: Moved the radio board over a little to give more room to solder.
Parts:
- moved U$15 0.48 mm to (77.2, 55.3)
Routing:
- net GND: vias 20 -> 22
